Commit message: アームを６軸に変更

File: turtlebot3_manipulation_description/ros2_control/turtlebot3_manipulation_system.ros2_control.xacro (robot description, xacro)
@@ -150,4 +150,28 @@
         </state_interface>
       </joint>
+      <joint name="${prefix}joint5">
+        <command_interface name="position">
+          <param name="min">${-pi*0.57}</param>
+          <param name="max">${pi*0.65}</param>
+        </command_interface>
+        <state_interface name="position">
+          <param name="initial_value">0.0</param>
+        </state_interface>
+        <state_interface name="velocity">
+          <param name="initial_value">0.0</param>
+        </state_interface>
+      </joint>
+      <joint name="${prefix}joint6">
+        <command_interface name="position">
+          <param name="min">${-pi*0.57}</param>
+          <param name="max">${pi*0.65}</param>
+        </command_interface>
+        <state_interface name="position">
+          <param name="initial_value">0.0</param>
+        </state_interface>
+        <state_interface name="velocity">
+          <param name="initial_value">0.0</param>
+        </state_interface>
+      </joint>
       <joint name="${prefix}gripper_left_joint">
         <command_interface name="position">

File: turtlebot3_manipulation_description/urdf/open_manipulator_x.urdf.xacro (robot description, xacro)
@@ -24,5 +24,5 @@
         </geometry>
       </collision>
-       <inertial>
+      <inertial>
         <origin xyz="3.0876154e-04 0.0000000e+00 -1.2176461e-04" />
         <mass value="7.9119962e-02" />
@@ -54,5 +54,5 @@
         </geometry>
       </collision>
-       <inertial>
+      <inertial>
         <origin xyz="-3.0184870e-04 5.4043684e-04 ${0.018 + 2.9433464e-02}" />
         <mass value="9.8406837e-02" />
@@ -67,5 +67,5 @@
       <origin xyz="0.0 0.0 0.0595" rpy="0 0 0"/>
       <axis xyz="0 1 0"/>
-      <limit velocity="4.8" effort="1" lower="${-pi*0.57}" upper="${pi*0.5}" />
+      <limit velocity="4.8" effort="1" lower="${-pi*0.65}" upper="${pi*0.67}" />
       <dynamics damping="0.1"/>
     </joint>
@@ -84,7 +84,7 @@
         </geometry>
       </collision>
-       <inertial>
-        <origin xyz="1.0308393e-02 3.7743363e-04 1.0170197e-01" />
-        <mass value="1.3850917e-01" />
+      <inertial>
+        <origin xyz="0 0 0" />
+        <mass value="0.131" />
         <inertia ixx="3.3055381e-04" ixy="-9.7940978e-08" ixz="-3.8505711e-05"
                  iyy="3.4290447e-04" iyz="-1.5717516e-06"
@@ -95,7 +95,7 @@
       <parent link="${prefix}link3"/>
       <child link="${prefix}link4"/>
-      <origin xyz="0.024 0 0.128" rpy="0 0 0"/>
-      <axis xyz="0 1 0"/>
-      <limit velocity="4.8" effort="1" lower="${-pi*0.3}" upper="${pi*0.44}" />
+      <origin xyz="0.0 0 0.124" rpy="0 0 0"/>
+      <axis xyz="0 1 0"/>
+      <limit velocity="4.8" effort="1" lower="${-pi*0.60}" upper="${pi*0.68}" />
       <dynamics damping="0.1"/>
     </joint>
@@ -114,10 +114,8 @@
         </geometry>
       </collision>
-       <inertial>
-        <origin xyz="9.0909590e-02 3.8929816e-04 2.2413279e-04" />
-        <mass value="1.3274562e-01" />
-        <inertia ixx="3.0654178e-05" ixy="-1.2764155e-06" ixz="-2.6874417e-07"
-                 iyy="2.4230292e-04" iyz="1.1559550e-08"
-                 izz="2.5155057e-04" />
+      <inertial>
+        <origin xyz="0 0 0" />
+        <mass value="0.098" />
+        <inertia ixx="0.1" ixy="0.0" ixz="0.0" iyy="0.1" iyz="0.0" izz="0.1" />
       </inertial>
     </link>
@@ -125,12 +123,12 @@
       <parent link="${prefix}link4"/>
       <child link="${prefix}link5"/>
-      <origin xyz="0.124 0.0 0.0" rpy="0 0 0"/>
-      <axis xyz="0 1 0"/>
-      <limit velocity="4.8" effort="1" lower="${-pi*0.57}" upper="${pi*0.65}" />
+      <origin xyz="0.0 0.0 0.045" rpy="0 0 0"/>
+      <axis xyz="0 0 1"/>
+      <limit velocity="4.8" effort="1" lower="${-pi*0.9}" upper="${pi*0.9}" />
       <dynamics damping="0.1"/>
     </joint>
     <link name="${prefix}link5">
       <visual>
-        <origin xyz="0 0 0" rpy="0 0 0"/>
+        <origin xyz="0 0 0.019" rpy="0 0 0"/>
         <geometry>
           <mesh filename="${meshes_file_direction}/link5.stl" scale="0.001 0.001 0.001"/>
@@ -139,10 +137,43 @@
       </visual>
       <collision>
-        <origin xyz="0 0 0" rpy="0 0 0"/>
+        <origin xyz="0 0 0.019" rpy="0 0 0"/>
         <geometry>
           <mesh filename="${meshes_file_direction}/link5.stl" scale="0.001 0.001 0.001"/>
         </geometry>
       </collision>
-       <inertial>
+      <inertial>
+        <origin xyz="0 0 0" />
+        <mass value="0.098" />
+        <inertia ixx="0.1" ixy="0.0" ixz="0.0" iyy="0.1" iyz="0.0" izz="0.1" />
+      </inertial>
+    </link>
+    <joint name="${prefix}joint5" type="revolute">
+      <parent link="${prefix}link5"/>
+      <child link="${prefix}link6"/>
+      <origin xyz="0.0 0.0 0.0595" rpy="0 0 0"/>
+      <axis xyz="0 1 0"/>
+      <limit velocity="4.8" effort="1" lower="${-pi*0.63}" upper="${pi*0.67}" />
+      <dynamics damping="0.1"/>
+    </joint>
+    <link name="${prefix}link6">
+      <visual>
+        <origin xyz="0 0 0.0" rpy="0 0 0"/>
+        <geometry>
+          <mesh filename="${meshes_file_direction}/link6.stl" scale="0.001 0.001 0.001"/>
+        </geometry>
+        <material name="grey"/>
+      </visual>
+      <collision>
+        <origin xyz="0 0 0.0" rpy="0 0 0"/>
+        <geometry>
+          <mesh filename="${meshes_file_direction}/link6.stl" scale="0.001 0.001 0.001"/>
+        </geometry>
+      </collision>
+      <inertial>
+        <origin xyz="0 0 0" />
+        <mass value="0.033" />
+        <inertia ixx="0.1" ixy="0.0" ixz="0.0" iyy="0.1" iyz="0.0" izz="0.1" />
+      </inertial>
+      <inertial>
         <origin xyz="4.4206755e-02 3.6839985e-07 8.9142216e-03" />
         <mass value="1.4327573e-01" />
@@ -152,24 +183,72 @@
       </inertial>
     </link>
+    <joint name="${prefix}joint6" type="revolute">
+      <parent link="${prefix}link6"/>
+      <child link="${prefix}link7"/>
+      <origin xyz="0.0 0.0 0.0475" rpy="0 0 0"/>
+      <axis xyz="0 0 1"/>
+      <limit velocity="4.8" effort="1" lower="${-pi*0.9}" upper="${pi*0.9}" />
+      <dynamics damping="0.1"/>
+    </joint>
+    <link name="${prefix}link7">
+      <visual>
+        <origin xyz="0 0 0.0" rpy="0 0 0"/>
+        <geometry>
+          <mesh filename="${meshes_file_direction}/link7.stl" scale="0.001 0.001 0.001"/>
+        </geometry>
+        <!-- <material name="grey"/> -->
+      </visual>
+      <collision>
+        <origin xyz="0 0 0.0" rpy="0 0 0"/>
+        <geometry>
+          <mesh filename="${meshes_file_direction}/link7.stl" scale="0.001 0.001 0.001"/>
+        </geometry>
+      </collision>
+      <inertial>
+        <origin xyz="4.4206755e-02 3.6839985e-07 8.9142216e-03" />
+        <mass value="1.4327573e-01" />
+        <inertia ixx="8.0870749e-05" ixy="0.0" ixz="-1.0157896e-06" iyy="7.5980465e-05" iyz="0.0" izz="9.3127351e-05" />
+      </inertial>
+    </link>
+    <link name="${prefix}gripper_left_link">
+      <visual>
+        <origin xyz="0 0 0" rpy="0 0 0"/>
+        <geometry>
+          <mesh filename="${meshes_file_direction}/gripper_left_palm.stl" scale="0.001 0.001 0.001"/>
+        </geometry>
+        <material name="grey"/>
+      </visual>
+      <collision>
+        <origin xyz="0 0 0" rpy="0 0 0"/>
+        <geometry>
+          <mesh filename="${meshes_file_direction}/gripper_left_palm.stl" scale="0.001 0.001 0.001"/>
+        </geometry>
+      </collision>
+      <inertial>
+        <origin xyz="0 0 0" />
+        <mass value="1.0e-03" />
+        <inertia ixx="1.0e-03" ixy="0.0" ixz="0.0" iyy="1.0e-03" iyz="0.0" izz="1.0e-03" />
+      </inertial>
+    </link>
     <joint name="${prefix}gripper_left_joint" type="prismatic">
-      <parent link="${prefix}link5"/>
+      <parent link="${prefix}link7"/>
       <child link="${prefix}gripper_left_link"/>
-      <origin xyz="0.0817 0.021 0.0" rpy="0 0 0"/>
+      <origin xyz="0.0 0.021 0.0707" rpy="0 0 0"/>
       <axis xyz="0 1 0"/>
       <limit velocity="4.8" effort="1" lower="-0.010" upper="0.019" />
       <dynamics damping="0.1"/>
     </joint>
-    <link name="${prefix}gripper_left_link">
-      <visual>
-        <origin xyz="0 0 0" rpy="0 0 0"/>
-        <geometry>
-          <mesh filename="${meshes_file_direction}/gripper_left_palm.stl" scale="0.001 0.001 0.001"/>
-        </geometry>
-        <material name="grey"/>
-      </visual>
-      <collision>
-        <origin xyz="0 0 0" rpy="0 0 0"/>
-        <geometry>
-          <mesh filename="${meshes_file_direction}/gripper_left_palm.stl" scale="0.001 0.001 0.001"/>
+    <link name="${prefix}gripper_right_link">
+      <visual>
+        <origin xyz="0 0 0" rpy="0 0 0"/>
+        <geometry>
+          <mesh filename="${meshes_file_direction}/gripper_right_palm.stl" scale="0.001 0.001 0.001"/>
+        </geometry>
+        <material name="grey"/>
+      </visual>
+      <collision>
+        <origin xyz="0 0 0" rpy="0 0 0"/>
+        <geometry>
+          <mesh filename="${meshes_file_direction}/gripper_right_palm.stl" scale="0.001 0.001 0.001"/>
         </geometry>
       </collision>
@@ -177,13 +256,11 @@
         <origin xyz="0 0 0" />
         <mass value="1.0e-03" />
-        <inertia ixx="1.0e-06" ixy="0.0" ixz="0.0"
-                 iyy="1.0e-06" iyz="0.0"
-                 izz="1.0e-06" />
+        <inertia ixx="1.0e-03" ixy="0.0" ixz="0.0" iyy="1.0e-03" iyz="0.0" izz="1.0e-03" />
       </inertial>
     </link>
     <joint name="${prefix}gripper_right_joint" type="prismatic">
-      <parent link="${prefix}link5"/>
+      <parent link="${prefix}link7"/>
       <child link="${prefix}gripper_right_link"/>
-      <origin xyz="0.0817 -0.021 0" rpy="0 0 0"/>
+      <origin xyz="0.0 -0.021 0.0707" rpy="0 0 0"/>
       <axis xyz="0 -1 0"/>
       <limit velocity="4.8" effort="1" lower="-0.010" upper="0.019" />
@@ -191,40 +268,30 @@
       <dynamics damping="0.1"/>
     </joint>
-    <link name="${prefix}gripper_right_link">
-      <visual>
-        <origin xyz="0 0 0" rpy="0 0 0"/>
-        <geometry>
-          <mesh filename="${meshes_file_direction}/gripper_right_palm.stl" scale="0.001 0.001 0.001"/>
-        </geometry>
-        <material name="grey"/>
-      </visual>
-      <collision>
-        <origin xyz="0 0 0" rpy="0 0 0"/>
-        <geometry>
-          <mesh filename="${meshes_file_direction}/gripper_right_palm.stl" scale="0.001 0.001 0.001"/>
-        </geometry>
-      </collision>
+    <joint name="${prefix}end_effector_joint" type="fixed">
+      <origin xyz="0.0 0.0 0.115" rpy="0 0 0"/>
+      <parent link="${prefix}link7"/>
+      <child link="${prefix}end_effector_link"/>
+    </joint>
+    <link name="${prefix}end_effector_link">
+      <visual>
+        <origin xyz="0 0 0" rpy="0 0 0"/>
+        <geometry>
+          <box size="0.01 0.01 0.01" />
+        </geometry>
+        <material name="grey"/>
+      </visual>
       <inertial>
         <origin xyz="0 0 0" />
         <mass value="1.0e-03" />
-        <inertia ixx="1.0e-06" ixy="0.0" ixz="0.0"
-                 iyy="1.0e-06" iyz="0.0"
-                 izz="1.0e-06" />
-      </inertial>
-    </link>
-    <joint name="${prefix}end_effector_joint" type="fixed">
-      <parent link="${prefix}link5"/>
-      <child link="${prefix}end_effector_link"/>
-      <origin xyz="0.126 0.0 0.0" rpy="0 0 0"/>
-    </joint>
-    <link name="${prefix}end_effector_link">
-      <visual>
-        <origin xyz="0 0 0" rpy="0 0 0"/>
-        <geometry>
-          <box size="0.01 0.01 0.01" />
-        </geometry>
-        <material name="red"/>
-       </visual>
-    </link>
+        <inertia ixx="1.0e-03" ixy="0.0" ixz="0.0" iyy="1.0e-03" iyz="0.0" izz="1.0e-03" />
+      </inertial>
+    </link>
+    <!-- Move it 2 not find mimic-->
+    <!-- https://github.com/ROBOTIS-GIT/turtlebot3_manipulation/issues/66  -->
+    <joint name="${prefix}gripper_right_joint_mimic" type="fixed">
+      <parent link="${prefix}link7" />
+      <child link="dummy_mimic_fix" />
+    </joint>
+    <link name="dummy_mimic_fix"/>
   </xacro:macro>
 </robot>
