Commit message: アームを６軸に変更

File: turtlebot3_manipulation_description/urdf/turtlebot3_waffle_pi.urdf.xacro (robot description, xacro)
@@ -6,190 +6,185 @@
 -->
 <robot xmlns:xacro="http://www.ros.org/wiki/xacro">
+  <xacro:include filename="$(find realsense2_description)/urdf/_d435.urdf.xacro"/>
   <xacro:macro name="turtlebot3_waffle_pi" params="prefix">
   <xacro:property
     name="meshes_file_direction"
     value="package://turtlebot3_manipulation_description/meshes/turtlebot3_waffle_pi"/>
-  <link name="${prefix}base_footprint"/>
-  <joint name="${prefix}base_joint" type="fixed">
-    <parent link="${prefix}base_footprint"/>
-    <child link="${prefix}base_link" />
-    <origin xyz="0 0 0.010" rpy="0 0 0"/>
-  </joint>
-  <link name="${prefix}base_link">
-    <visual>
-      <origin xyz="-0.064 0 0.0" rpy="0 0 0"/>
-      <geometry>
-        <mesh filename="${meshes_file_direction}/base.stl" scale="0.001 0.001 0.001"/>
-      </geometry>
-      <material name="light_black"/>
-    </visual>
-    <collision>
-      <origin xyz="-0.064 0 0.047" rpy="0 0 0"/>
-      <geometry>
-        <box size="0.266 0.266 0.094"/>
-      </geometry>
-    </collision>
-    <inertial>
-      <origin xyz="0 0 0" rpy="0 0 0"/>
-      <mass value="1.3729096e+00"/>
+    <link name="${prefix}base_footprint"/>
+    <joint name="${prefix}base_joint" type="fixed">
+      <parent link="${prefix}base_footprint"/>
+      <child link="${prefix}base_link" />
+      <origin xyz="0 0 0.060" rpy="0 0 0"/>
+    </joint>
+    <link name="${prefix}base_link">
+      <visual>
+        <origin xyz="0 0 0" rpy="0 0 0"/>
+        <geometry>
+          <mesh filename="${meshes_file_direction}/base.stl" scale="0.001 0.001 0.001"/>
+        </geometry>
+        <material name="light_black"/>
+      </visual>
+      <collision>
+        <origin xyz="-0.065 0 0.0225" rpy="0 0 0"/>
+        <geometry>
+          <box size="0.266 0.266 0.095"/>
+        </geometry>
+      </collision>
+      <inertial>
+        <origin xyz="0 0 0" rpy="0 0 0"/>
+        <mass value="1.3729096e+00"/>
       <inertia ixx="8.7002718e-03" ixy="-4.7576583e-05" ixz="1.1160499e-04"
                iyy="8.6195418e-03" iyz="-3.5422299e-06"
                izz="1.4612727e-02" />
-    </inertial>
-  </link>
-  <joint name="${prefix}wheel_left_joint" type="continuous">
-    <parent link="${prefix}base_link"/>
-    <child link="${prefix}wheel_left_link"/>
-    <origin xyz="0.0 0.144 0.023" rpy="-1.57 0 0"/>
-    <axis xyz="0 0 1"/>
-  </joint>
-  <link name="${prefix}wheel_left_link">
-    <visual>
-      <origin xyz="0 0 0" rpy="1.57 0 0"/>
-      <geometry>
-        <mesh filename="${meshes_file_direction}/left_tire.stl" scale="0.001 0.001 0.001"/>
-      </geometry>
-      <material name="dark"/>
-    </visual>
-    <collision>
-      <origin xyz="0 0 0" rpy="0 0 0"/>
-      <geometry>
-        <cylinder length="0.018" radius="0.033"/>
-      </geometry>
-    </collision>
-    <inertial>
-      <origin xyz="0 0 0" />
-      <mass value="2.8498940e-02" />
+      </inertial>
+    </link>
+    <joint name="${prefix}wheel_left_joint" type="continuous">
+      <parent link="${prefix}base_link"/>
+      <child link="${prefix}wheel_left_link"/>
+      <origin xyz="0.0 0.147125 0.0" rpy="-1.57 0 0"/>
+      <axis xyz="0 0 1"/>
+    </joint>
+    <link name="${prefix}wheel_left_link">
+      <visual>
+        <origin xyz="0 0 0" rpy="1.57 0 0"/>
+        <geometry>
+          <mesh filename="${meshes_file_direction}/tire.stl" scale="0.001 0.001 0.001"/>
+        </geometry>
+        <material name="dark"/>
+      </visual>
+      <collision>
+        <origin xyz="0 0 0" rpy="0 0 0"/>
+        <geometry>
+          <cylinder length="0.02425" radius="0.06"/>
+        </geometry>
+      </collision>
+      <inertial>
+        <origin xyz="0 0 0" />
+        <mass value="2.8498940e-02" />
       <inertia ixx="1.1175580e-05" ixy="-4.2369783e-11" ixz="-5.9381719e-09"
                iyy="1.1192413e-05" iyz="-1.4400107e-11"
                izz="2.0712558e-05" />
       </inertial>
-  </link>
-  <joint name="${prefix}wheel_right_joint" type="continuous">
-    <parent link="${prefix}base_link"/>
-    <child link="${prefix}wheel_right_link"/>
-    <origin xyz="0.0 -0.144 0.023" rpy="-1.57 0 0"/>
-    <axis xyz="0 0 1"/>
-  </joint>
-  <link name="${prefix}wheel_right_link">
-    <visual>
-      <origin xyz="0 0 0" rpy="1.57 0 0"/>
-      <geometry>
-        <mesh filename="${meshes_file_direction}/right_tire.stl" scale="0.001 0.001 0.001"/>
-      </geometry>
-      <material name="dark"/>
-    </visual>
-    <collision>
-      <origin xyz="0 0 0" rpy="0 0 0"/>
-      <geometry>
-        <cylinder length="0.018" radius="0.033"/>
-      </geometry>
-    </collision>
-    <inertial>
-      <origin xyz="0 0 0" />
-      <mass value="2.8498940e-02" />
+    </link>
+    <joint name="${prefix}wheel_right_joint" type="continuous">
+      <parent link="${prefix}base_link"/>
+      <child link="${prefix}wheel_right_link"/>
+      <origin xyz="0.0 -0.147125 0.0" rpy="-1.57 0 0"/>
+      <axis xyz="0 0 1"/>
+    </joint>
+    <link name="${prefix}wheel_right_link">
+      <visual>
+        <origin xyz="0 0 0" rpy="1.57 0 0"/>
+        <geometry>
+          <mesh filename="${meshes_file_direction}/tire.stl" scale="0.001 0.001 0.001"/>
+        </geometry>
+        <material name="dark"/>
+      </visual>
+      <collision>
+        <origin xyz="0 0 0" rpy="0 0 0"/>
+        <geometry>
+          <cylinder length="0.02425" radius="0.06"/>
+        </geometry>
+      </collision>
+      <inertial>
+        <origin xyz="0 0 0" />
+        <mass value="2.8498940e-02" />
       <inertia ixx="1.1175580e-05" ixy="-4.2369783e-11" ixz="-5.9381719e-09"
                iyy="1.1192413e-05" iyz="-1.4400107e-11"
                izz="2.0712558e-05" />
       </inertial>
-  </link>
-  <joint name="${prefix}caster_back_right_joint" type="fixed">
-    <parent link="${prefix}base_link"/>
-    <child link="${prefix}caster_back_right_link"/>
-    <origin xyz="-0.177 -0.064 -0.004" rpy="-1.57 0 0"/>
-  </joint>
-  <link name="${prefix}caster_back_right_link">
-    <collision>
-      <origin xyz="0 0.001 0" rpy="0 0 0"/>
-      <geometry>
-        <box size="0.030 0.009 0.020"/>
-      </geometry>
-    </collision>
-    <inertial>
-      <origin xyz="0 0 0" />
-      <mass value="0.005" />
-      <inertia ixx="0.001" ixy="0.0" ixz="0.0"
-               iyy="0.001" iyz="0.0"
-               izz="0.001" />
-    </inertial>
-  </link>
-  <joint name="${prefix}caster_back_left_joint" type="fixed">
-    <parent link="${prefix}base_link"/>
-    <child link="${prefix}caster_back_left_link"/>
-    <origin xyz="-0.177 0.064 -0.004" rpy="-1.57 0 0"/>
-  </joint>
-  <link name="${prefix}caster_back_left_link">
-    <collision>
-      <origin xyz="0 0.001 0" rpy="0 0 0"/>
-      <geometry>
-        <box size="0.030 0.009 0.020"/>
-      </geometry>
-    </collision>
-    <inertial>
-      <origin xyz="0 0 0" />
-      <mass value="0.005" />
-      <inertia ixx="0.001" ixy="0.0" ixz="0.0"
-               iyy="0.001" iyz="0.0"
-               izz="0.001" />
-    </inertial>
-  </link>
-  <joint name="${prefix}imu_joint" type="fixed">
-    <parent link="${prefix}base_link"/>
-    <child link="${prefix}imu_link"/>
-    <origin xyz="0.0 0 0.068" rpy="0 0 0"/>
-  </joint>
-  <link name="${prefix}imu_link"/>
-  <joint name="${prefix}scan_joint" type="fixed">
-    <parent link="${prefix}base_link"/>
-    <child link="${prefix}base_scan"/>
-    <origin xyz="-0.024 0 0.122" rpy="0 0 0"/>
-  </joint>
-  <link name="${prefix}base_scan">
-    <visual>
-      <origin xyz="0 0 0.0" rpy="0 0 0"/>
-      <geometry>
-        <mesh filename="${meshes_file_direction}/ladar.stl" scale="0.001 0.001 0.001"/>
-      </geometry>
-      <material name="dark"/>
-    </visual>
-    <collision>
-      <origin xyz="0.015 0 -0.0065" rpy="0 0 0"/>
-      <geometry>
-        <cylinder length="0.0315" radius="0.055"/>
-      </geometry>
-    </collision>
-    <inertial>
-      <mass value="0.114" />
-      <origin xyz="0 0 0" />
-      <inertia ixx="0.001" ixy="0.0" ixz="0.0"
-               iyy="0.001" iyz="0.0"
-               izz="0.001" />
-    </inertial>
-  </link>
-  <joint name="${prefix}camera_joint" type="fixed">
-    <parent link="${prefix}base_link"/>
-    <child link="${prefix}camera_link"/>
-    <origin xyz="0.073 -0.011 0.084" rpy="0 0 0"/>
-  </joint>
-  <link name="${prefix}camera_link">
-    <collision>
-      <origin xyz="0.005 0.011 0.013" rpy="0 0 0"/>
-      <geometry>
-        <box size="0.015 0.030 0.027"/>
-      </geometry>
-    </collision>
-  </link>
-  <joint name="${prefix}camera_rgb_joint" type="fixed">
-    <parent link="${prefix}camera_link"/>
-    <child link="${prefix}camera_rgb_frame"/>
-    <origin xyz="0.003 0.011 0.009" rpy="0 0 0"/>
-  </joint>
-  <link name="${prefix}camera_rgb_frame"/>
-  <joint name="${prefix}camera_rgb_optical_joint" type="fixed">
-    <parent link="${prefix}camera_rgb_frame"/>
-    <child link="${prefix}camera_rgb_optical_frame"/>
-    <origin xyz="0 0 0" rpy="-1.57 0 -1.57"/>
-  </joint>
-  <link name="${prefix}camera_rgb_optical_frame"/>
+    </link>
+    <joint name="${prefix}caster_back_right_joint" type="fixed">
+      <parent link="${prefix}base_link"/>
+      <child link="${prefix}caster_back_right_link"/>
+      <origin xyz="-0.176 -0.064 -0.0556125" rpy="-1.57 0 0"/>
+    </joint>
+    <link name="${prefix}caster_back_right_link">
+      <collision>
+        <geometry>
+          <box size="0.030 0.009 0.005"/>
+        </geometry>
+      </collision>
+      <visual>
+        <geometry>
+          <sphere radius="0.005"/>
+        </geometry>
+        <material name="dark"/>
+      </visual>
+      <inertial>
+        <origin xyz="0 0 0" />
+        <mass value="0.005" />
+        <inertia ixx="0.001" ixy="0.0" ixz="0.0" iyy="0.001" iyz="0.0" izz="0.001" />
+      </inertial>
+    </link>
+    <joint name="${prefix}caster_back_left_joint" type="fixed">
+      <parent link="${prefix}base_link"/>
+      <child link="${prefix}caster_back_left_link"/>
+      <origin xyz="-0.176 0.064 -0.0556125" rpy="-1.57 0 0"/>
+    </joint>
+    <link name="${prefix}caster_back_left_link">
+      <collision>
+        <geometry>
+          <box size="0.030 0.009 0.005"/>
+        </geometry>
+      </collision>
+      <visual>
+        <geometry>
+          <sphere radius="0.005"/>
+        </geometry>
+        <material name="dark"/>
+      </visual>
+      <inertial>
+        <origin xyz="0 0 0" />
+        <mass value="0.005" />
+        <inertia ixx="0.001" ixy="0.0" ixz="0.0" iyy="0.001" iyz="0.0" izz="0.001" />
+      </inertial>
+    </link>
+    <joint name="${prefix}imu_joint" type="fixed">
+      <parent link="${prefix}base_link"/>
+      <child link="${prefix}imu_link"/>
+      <origin xyz="0.0 0 0.033" rpy="0 0 0"/>
+    </joint>
+    <link name="${prefix}imu_link"/>
+    <joint name="${prefix}scan_joint" type="fixed">
+      <parent link="${prefix}base_link"/>
+      <child link="${prefix}base_scan"/>
+      <origin xyz="0.027 0 0.10045" rpy="0 0 0"/>
+    </joint>
+    <link name="${prefix}base_scan">
+      <visual>
+        <origin xyz="0 0 0" rpy="0 0 0"/>
+        <geometry>
+          <mesh filename="${meshes_file_direction}/ladar.stl" scale="0.001 0.001 0.001"/>
+        </geometry>
+        <material name="dark"/>
+      </visual>
+      <collision>
+        <origin xyz="0.0 0 -0.0065" rpy="0 0 0"/>
+        <geometry>
+          <cylinder length="0.0315" radius="0.055"/>
+        </geometry>
+      </collision>
+      <inertial>
+        <mass value="0.114" />
+        <origin xyz="0 0 0" />
+        <inertia ixx="0.001" ixy="0.0" ixz="0.0" iyy="0.001" iyz="0.0" izz="0.001" />
+      </inertial>
+    </link>
+    <joint name="${prefix}battery_joint" type="fixed">
+      <parent link="${prefix}base_link"/>
+      <child link="${prefix}battery_link"/>
+      <origin xyz="-0.08 0 0" rpy="0 0 0"/>
+    </joint>
+    <link name="${prefix}battery_link">
+      <inertial>
+        <mass value="1.5" />
+        <origin xyz="0 0 0" />
+        <inertia ixx="0.001" ixy="0.0" ixz="0.0" iyy="0.001" iyz="0.0" izz="0.001" />
+      </inertial>
+    </link>
+    <xacro:sensor_d435 parent="base_link" use_nominal_extrinsics="false" add_plug="false" use_mesh="true">
+      <origin xyz="0.04855 -0.0175 -0.0142" rpy="0 0 0"/>
+    </xacro:sensor_d435>
   </xacro:macro>
 </robot>
