Commit message: アームの位置を修正

File: turtlebot3_manipulation_description/urdf/turtlebot3_manipulation.urdf.xacro (robot description, xacro)
@@ -24,5 +24,5 @@
     <parent link="$(arg prefix)base_link"/>
     <child link="$(arg prefix)link1"/>
-    <origin xyz="-0.092 0.0 0.091" rpy="0 0 0"/>
+    <origin xyz="-0.036 0.0 0.07" rpy="0 0 0"/>
   </joint>
   <xacro:open_manipulator_x prefix="$(arg prefix)" />
